File: caphumidsens_rev4_rc2.brd (EAGLE design)
At the start: 110 x 9 mm, 9 parts, among them IC1 555

Commit message: preparing rev4-final
Parts:
- moved R1 0.25 mm to (11.5, 6.75)
Routing:
- net N$1: track 24.3 -> 25.0 mm
- net VCC: track 35.1 -> 35.7 mm
Other:
- board text added: "projects@carwe.de"
- board text removed: "info@carwe.de"
Changed lines of the file:
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@@
 <layer number="20" name="Dimension" color="15" fill="1" visible="yes" active="yes"/>
 <layer number="21" name="tPlace" color="7" fill="1" visible="yes" active="yes"/>
-<layer number="22" name="bPlace" color="7" fill="1" visible="yes" active="yes"/>
-<layer number="23" name="tOrigins" color="15" fill="1" visible="no" active="yes"/>
+<layer number="22" name="bPlace" color="7" fill="1" visible="no" active="yes"/>
+<layer number="23" name="tOrigins" color="15" fill="1" visible="yes" active="yes"/>
 <layer number="24" name="bOrigins" color="15" fill="1" visible="no" active="yes"/>
 <layer number="25" name="tNames" color="7" fill="1" visible="yes" active="yes"/>
@@
 <layer number="28" name="bValues" color="7" fill="1" visible="no" active="yes"/>
 <layer number="29" name="tStop" color="7" fill="3" visible="yes" active="yes"/>
-<layer number="30" name="bStop" color="7" fill="6" visible="yes" active="yes"/>
+<layer number="30" name="bStop" color="7" fill="6" visible="no" active="yes"/>
 <layer number="31" name="tCream" color="7" fill="4" visible="no" active="yes"/>
 <layer number="32" name="bCream" color="7" fill="5" visible="no" active="yes"/>
@@
 <text x="8.7" y="5.9" size="0.8128" layer="25" font="vector" ratio="20">C1</text>
 <text x="8.5" y="2.9" size="0.8128" layer="25" font="vector" ratio="20">C2</text>
-<text x="10.85" y="4.35" size="0.8128" layer="25" font="vector" ratio="20">R1</text>
-<text x="10.85" y="0.75" size="0.8128" layer="25" font="vector" ratio="20">R2</text>
+<text x="10.85" y="4.45" size="0.8128" layer="25" font="vector" ratio="20">R1</text>
+<text x="10.85" y="0.7" size="0.8128" layer="25" font="vector" ratio="20">R2</text>
 <text x="7.2" y="1.7" size="0.8128" layer="25" font="vector" ratio="20" rot="R180">D1</text>
 <text x="2.9" y="3.9" size="0.8128" layer="25" font="vector" ratio="20">IC1</text>
@@
 <text x="32" y="2" size="0.8128" layer="25" font="vector" ratio="15" rot="R180">IC1=NE555/TLC555</text>
 <text x="53" y="5.2" size="0.8128" layer="25" font="vector" ratio="15" rot="R180">caphumidsens rev4</text>
-<text x="51" y="3.8" size="0.8128" layer="25" font="vector" ratio="15" rot="R180">info@carwe.de</text>
+<text x="52.65" y="4" size="0.8128" layer="25" font="vector" ratio="15" rot="R180">projects@carwe.de</text>
 </plain>
 <attributes>
@@
 <elements>
 <element name="IC1" library="linear" package="SO08" value="555" x="3" y="4.5" smashed="yes"/>
-<element name="R1" library="SparkFun" package="0805" value="" x="11.5" y="6.5" smashed="yes" rot="R90">
-<attribute name="VALUE" x="12.897" y="5.484" size="0.4064" layer="27" rot="R90"/>
+<element name="R1" library="SparkFun" package="0805" value="" x="11.5" y="6.75" smashed="yes" rot="R90">
+<attribute name="VALUE" x="12.897" y="5.734" size="0.4064" layer="27" rot="R90"/>
 </element>
 <element name="R2" library="SparkFun" package="0805" value="" x="11.5" y="3" smashed="yes" rot="R90">
@@
 </element>
 <element name="GND" library="wirepad" package="SMD1,27-2,54" value="WIREPADSMD2,54-5,08" x="4.1" y="4.5" smashed="yes" rot="MR90">
-<attribute name="NAME" x="1.8" y="3.5" size="0.8128" layer="26" font="vector" ratio="20" rot="SMR90"/>
+<attribute name="NAME" x="1.8" y="3.4" size="0.8128" layer="26" font="vector" ratio="20" rot="SMR90"/>
 </element>
 <element name="D1" library="seb" package="DIODE_0805" value="DIODE_0805" x="8.5" y="1.5" smashed="yes" rot="R180"/>
@@
 <contactref element="IC1" pad="7"/>
 <contactref element="D1" pad="2"/>
-<wire x1="11.5" y1="5.6" x2="11.5" y2="3.9" width="0.4064" layer="1"/>
-<wire x1="9" y1="3" x2="10.6" y2="3" width="0.4064" layer="1"/>
-<wire x1="10.6" y1="3" x2="11.5" y2="3.9" width="0.4064" layer="1"/>
+<wire x1="11.5" y1="5.85" x2="11.5" y2="3.9" width="0.4064" layer="1"/>
+<wire x1="9" y1="3" x2="11.1" y2="3" width="0.4064" layer="1"/>
 <via x="1.1" y="4.5" extent="1-16" drill="0.3302"/>
 <via x="12.7" y="5.5" extent="1-16" drill="0.3302"/>
-<wire x1="12.7" y1="5.5" x2="11.6" y2="5.5" width="0.4064" layer="1"/>
-<wire x1="11.6" y1="5.5" x2="11.5" y2="5.6" width="0.4064" layer="1"/>
 <wire x1="2.365" y1="7.1" x2="2.365" y2="5.065" width="0.4064" layer="1"/>
 <wire x1="9" y1="3" x2="7.6" y2="1.6" width="0.4064" layer="1"/>
@@
 <wire x1="2.365" y1="5.065" x2="1.8" y2="4.5" width="0.4064" layer="1"/>
 <wire x1="1.8" y1="4.5" x2="1.1" y2="4.5" width="0.4064" layer="1"/>
+<wire x1="11.5" y1="5.85" x2="12.35" y2="5.85" width="0.4064" layer="1"/>
+<wire x1="12.35" y1="5.85" x2="12.7" y2="5.5" width="0.4064" layer="1"/>
+<wire x1="11.1" y1="3" x2="11.5" y2="3.4" width="0.4064" layer="1"/>
+<wire x1="11.5" y1="3.4" x2="11.5" y2="3.9" width="0.4064" layer="1"/>
 </signal>
 <signal name="VCC">
@@
 <contactref element="VCC" pad="1"/>
 <wire x1="4.905" y1="1.9" x2="4.905" y2="1.905" width="0.4064" layer="1"/>
-<wire x1="11.5" y1="7.4" x2="10.9" y2="7.4" width="0.4064" layer="1"/>
-<wire x1="10.9" y1="7.4" x2="10.5" y2="7" width="0.4064" layer="1"/>
-<wire x1="10.5" y1="7" x2="10.5" y2="6.5" width="0.4064" layer="1"/>
+<wire x1="10.5" y1="7.35" x2="10.5" y2="6.5" width="0.4064" layer="1"/>
 <wire x1="10.5" y1="6.5" x2="9.4" y2="5.4" width="0.4064" layer="1"/>
 <wire x1="9.4" y1="5.4" x2="9.4" y2="4.5" width="0.4064" layer="1"/>
@@
 <via x="1.1" y="5.45" extent="1-16" drill="0.3302"/>
 <via x="12.7" y="7.5" extent="1-16" drill="0.3302"/>
-<wire x1="12.7" y1="7.5" x2="11.6" y2="7.5" width="0.4064" layer="1"/>
-<wire x1="11.6" y1="7.5" x2="11.5" y2="7.4" width="0.4064" layer="1"/>
+<wire x1="11.6" y1="7.5" x2="11.5" y2="7.65" width="0.4064" layer="1"/>
 <wire x1="1.1" y1="7.1" x2="1.5" y2="7.5" width="0.4064" layer="16"/>
 <wire x1="12.7" y1="7.5" x2="13.95" y2="7.5" width="0.4064" layer="16"/>
@@
 <wire x1="7.8" y1="3" x2="7" y2="3" width="0.4064" layer="1"/>
 <wire x1="5.9" y1="1.9" x2="7" y2="3" width="0.4064" layer="1"/>
+<wire x1="10.5" y1="7.35" x2="10.8" y2="7.65" width="0.4064" layer="1"/>
+<wire x1="10.8" y1="7.65" x2="11.5" y2="7.65" width="0.4064" layer="1"/>
+<wire x1="12.7" y1="7.5" x2="12.55" y2="7.65" width="0.4064" layer="1"/>
+<wire x1="12.55" y1="7.65" x2="11.5" y2="7.65" width="0.4064" layer="1"/>
 </signal>
 <signal name="N$3">
