File: caphumidsens2_rev1_rc3.brd (EAGLE design)
At the start: 110 x 10 mm, 12 parts, among them IC1 ATtiny25/45/85

Commit message: finetuning, misc
Routing:
- net 2_3RD_VCC_VREF: track 19.3 -> 18.6 mm
Changed lines of the file:
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@@
 <wire x1="8.4" y1="8.4" x2="9.45" y2="8.4" width="0.4064" layer="1"/>
 <wire x1="8.4" y1="8.4" x2="7.9" y2="8.5" width="0.4064" layer="1"/>
-<wire x1="7.9" y1="8.5" x2="7.2" y2="8.5" width="0.4064" layer="1"/>
-<via x="7.2" y="8.5" extent="1-16" drill="0.3302"/>
+<wire x1="7.9" y1="8.5" x2="7.3" y2="8.5" width="0.4064" layer="1"/>
+<via x="7.3" y="8.5" extent="1-16" drill="0.3302"/>
 <contactref element="OSC1" pad="4"/>
 <contactref element="OSC1" pad="4"/>
@@
 <wire x1="3" y1="8" x2="4.5" y2="8" width="0.4064" layer="16"/>
 <wire x1="4.5" y1="8" x2="5" y2="8.5" width="0.4064" layer="16"/>
-<wire x1="5" y1="8.5" x2="7.2" y2="8.5" width="0.4064" layer="16"/>
+<wire x1="5" y1="8.5" x2="7.3" y2="8.5" width="0.4064" layer="16"/>
 <wire x1="12.675" y1="4.575" x2="12.675" y2="5.2" width="0.4064" layer="1"/>
 <wire x1="12.675" y1="5.2" x2="12.075" y2="5.7" width="0.4064" layer="1"/>
@@
 <wire x1="12.5" y1="6.6" x2="13.5" y2="5.6" width="0.4064" layer="1"/>
 <wire x1="13.5" y1="5.6" x2="13.5" y2="1.5" width="0.4064" layer="1"/>
-<wire x1="6.2" y1="1.5" x2="6.8" y2="1.5" width="0.4064" layer="1"/>
+<wire x1="6.2" y1="1.5" x2="6.7" y2="1.5" width="0.4064" layer="1"/>
 <wire x1="7.7" y1="1.5" x2="9.5" y2="1.5" width="0.4064" layer="1"/>
-<wire x1="6.8" y1="1.5" x2="7.7" y2="1.5" width="0.4064" layer="1"/>
+<wire x1="6.7" y1="1.5" x2="7.7" y2="1.5" width="0.4064" layer="1"/>
 <wire x1="9.5" y1="1.5" x2="11.125" y2="1.5" width="0.4064" layer="1"/>
 <wire x1="11.125" y1="1.5" x2="13.5" y2="1.5" width="0.4064" layer="1"/>
 <wire x1="6.2" y1="1.5" x2="5.895" y2="1.805" width="0.4064" layer="1"/>
-<wire x1="3" y1="2" x2="6.4" y2="2" width="0.4064" layer="16"/>
-<wire x1="6.4" y1="2" x2="6.8" y2="1.5" width="0.4064" layer="16"/>
-<via x="6.8" y="1.5" extent="1-16" drill="0.3302"/>
+<wire x1="3" y1="2" x2="6.3" y2="2" width="0.4064" layer="16"/>
+<wire x1="6.3" y1="2" x2="6.7" y2="1.5" width="0.4064" layer="16"/>
+<via x="6.7" y="1.5" extent="1-16" drill="0.3302"/>
 <wire x1="11.125" y1="2.425" x2="11.125" y2="1.5" width="0.4064" layer="1"/>
 <contactref element="IC1" pad="4"/>
@@
 <wire x1="8.4" y1="5.6" x2="9.5" y2="4.5" width="0.4064" layer="1"/>
 <wire x1="9.5" y1="4.5" x2="9.5" y2="4.3" width="0.4064" layer="1"/>
-<wire x1="7.2" y1="6.5" x2="7.1" y2="6.6" width="0.4064" layer="16"/>
-<wire x1="7.1" y1="6.6" x2="15.7" y2="6.6" width="0.4064" layer="16"/>
-<wire x1="14.5" y1="6.6" x2="15.7" y2="6.6" width="0.4064" layer="1"/>
-<via x="15.7" y="6.6" extent="1-16" drill="0.3302"/>
-<via x="7.2" y="6.5" extent="1-16" drill="0.3302"/>
+<wire x1="7.3" y1="6.6" x2="15.6" y2="6.6" width="0.4064" layer="16"/>
+<wire x1="14.5" y1="6.6" x2="15.6" y2="6.6" width="0.4064" layer="1"/>
+<via x="15.6" y="6.6" extent="1-16" drill="0.3302"/>
+<via x="7.3" y="6.6" extent="1-16" drill="0.3302"/>
 <wire x1="8.4" y1="5.6" x2="8.4" y2="6.6" width="0.4064" layer="1"/>
-<wire x1="7.2" y1="6.5" x2="7.1" y2="6.6" width="0.4064" layer="1"/>
-<wire x1="7.1" y1="6.6" x2="8.4" y2="6.6" width="0.4064" layer="1"/>
-<wire x1="3.365" y1="6.35" x2="3.565" y2="6.5" width="0.4064" layer="16"/>
-<wire x1="3.565" y1="6.5" x2="7.2" y2="6.5" width="0.4064" layer="16"/>
+<wire x1="3.365" y1="6.35" x2="7.05" y2="6.35" width="0.4064" layer="16"/>
+<wire x1="7.05" y1="6.35" x2="7.3" y2="6.6" width="0.4064" layer="16"/>
+<wire x1="7.3" y1="6.6" x2="8.4" y2="6.6" width="0.4064" layer="1"/>
 </signal>
 <signal name="1_3RD_VCC_VREF">
@@
 <vertex x="99" y="9"/>
 </polygon>
-<wire x1="6.8" y1="7.5" x2="17" y2="7.5" width="0.4064" layer="16"/>
+<wire x1="6.7" y1="7.5" x2="17" y2="7.5" width="0.4064" layer="16"/>
 <wire x1="17" y1="7.5" x2="37" y2="7.5" width="0.4064" layer="16"/>
-<via x="6.8" y="7.5" extent="1-16" drill="0.3302"/>
+<via x="6.7" y="7.5" extent="1-16" drill="0.3302"/>
 <contactref element="R4" pad="1"/>
 <wire x1="17" y1="3.4" x2="17" y2="7.5" width="0.4064" layer="16"/>
-<wire x1="6.8" y1="7.5" x2="5.905" y2="7.5" width="0.4064" layer="1"/>
+<wire x1="6.7" y1="7.5" x2="5.905" y2="7.5" width="0.4064" layer="1"/>
 <wire x1="5.905" y1="7.5" x2="5.905" y2="7.654" width="0.4064" layer="1"/>
-<via x="15.7" y="2.6" extent="1-16" drill="0.3302"/>
-<wire x1="15.7" y1="2.6" x2="14.5" y2="2.6" width="0.4064" layer="1"/>
+<via x="15.6" y="2.6" extent="1-16" drill="0.3302"/>
+<wire x1="15.6" y1="2.6" x2="14.5" y2="2.6" width="0.4064" layer="1"/>
 <wire x1="17" y1="3.4" x2="16.2" y2="2.6" width="0.4064" layer="16"/>
-<wire x1="16.2" y1="2.6" x2="15.7" y2="2.6" width="0.4064" layer="16"/>
+<wire x1="16.2" y1="2.6" x2="15.6" y2="2.6" width="0.4064" layer="16"/>
 </signal>
 <signal name="CLOCK_IN">
@@
 <via x="3.355" y="3.65" extent="1-16" drill="0.3302"/>
 <wire x1="3.355" y1="2.346" x2="3.355" y2="3.65" width="0.4064" layer="1"/>
-<via x="12.675" y="3.47" extent="1-16" drill="0.3302"/>
-<wire x1="12.675" y1="3.47" x2="12.3" y2="3.65" width="0.4064" layer="16"/>
+<via x="12.675" y="3.42" extent="1-16" drill="0.3302"/>
+<wire x1="12.675" y1="3.42" x2="12.3" y2="3.65" width="0.4064" layer="16"/>
 <wire x1="12.3" y1="3.65" x2="3.355" y2="3.65" width="0.4064" layer="16"/>
-<wire x1="12.675" y1="3.47" x2="12.675" y2="2.425" width="0.4064" layer="1"/>
+<wire x1="12.675" y1="3.42" x2="12.675" y2="2.425" width="0.4064" layer="1"/>
 </signal>
 <signal name="OUTPUT_OR_DEBUGWIRE">
@@
 <contactref element="IC1" pad="6"/>
 <contactref element="R4" pad="2"/>
-<wire x1="15.7" y1="4.6" x2="6" y2="4.6" width="0.4064" layer="16"/>
-<wire x1="14.5" y1="4.4" x2="15.7" y2="4.4" width="0.4064" layer="1"/>
-<via x="15.7" y="4.4" extent="1-16" drill="0.3302"/>
-<wire x1="15.7" y1="4.4" x2="15.7" y2="4.6" width="0.4064" layer="16"/>
+<wire x1="15.6" y1="4.6" x2="6" y2="4.6" width="0.4064" layer="16"/>
+<wire x1="14.5" y1="4.4" x2="15.6" y2="4.4" width="0.4064" layer="1"/>
+<via x="15.6" y="4.4" extent="1-16" drill="0.3302"/>
+<wire x1="15.6" y1="4.4" x2="15.6" y2="4.6" width="0.4064" layer="16"/>
 <wire x1="6" y1="4.6" x2="5.54890625" y2="4.6" width="0.4064" layer="1"/>
 <wire x1="5.54890625" y1="4.6" x2="4.635" y2="5.51390625" width="0.4064" layer="1"/>

Commit message: finetuning, misc
Parts:
- IC1: value ATtiny25/45/85 -> ATtiny25/45/85/13A
- moved R4 0.20 mm to (14.7, 3.50)
Other:
- board text added: "IC1=ATtiny25/45/85/13A"
- board text removed: "IC1=ATtiny25/45/85"
Changed lines of the file:
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@@
 <layer number="19" name="Unrouted" color="6" fill="1" visible="yes" active="yes"/>
 <layer number="20" name="Dimension" color="15" fill="1" visible="yes" active="yes"/>
-<layer number="21" name="tPlace" color="7" fill="1" visible="no" active="yes"/>
-<layer number="22" name="bPlace" color="7" fill="1" visible="no" active="yes"/>
-<layer number="23" name="tOrigins" color="15" fill="1" visible="yes" active="yes"/>
+<layer number="21" name="tPlace" color="7" fill="1" visible="yes" active="yes"/>
+<layer number="22" name="bPlace" color="7" fill="1" visible="yes" active="yes"/>
+<layer number="23" name="tOrigins" color="15" fill="1" visible="no" active="yes"/>
 <layer number="24" name="bOrigins" color="15" fill="1" visible="no" active="yes"/>
 <layer number="25" name="tNames" color="7" fill="1" visible="yes" active="yes"/>
@@
 <wire x1="0" y1="10" x2="0" y2="0" width="0" layer="20"/>
 <wire x1="1.45" y1="1.2" x2="2.6" y2="1.2" width="0.4064" layer="25"/>
-<text x="19.5" y="5" size="0.8128" layer="25" font="vector" ratio="15">caphumidsens2 rev1</text>
-<text x="19.5" y="3.5" size="0.8128" layer="25" font="vector" ratio="15">projects@carwe.de</text>
+<text x="19.5" y="6.5" size="0.8128" layer="1" font="vector" ratio="15">caphumidsens2 rev1</text>
+<text x="19.5" y="5" size="0.8128" layer="1" font="vector" ratio="15">projects@carwe.de</text>
 <text x="37" y="6" size="0.8128" layer="25" font="vector" ratio="15">R1=R2=R3=100kOhm</text>
 <text x="37" y="5" size="0.8128" layer="25" font="vector" ratio="15">R4=</text>
 <text x="37" y="4" size="0.8128" layer="25" font="vector" ratio="15">C1=100nF, C2=C3=10nF</text>
-<text x="37" y="3" size="0.8128" layer="25" font="vector" ratio="15">IC1=ATtiny25/45/85</text>
+<text x="37" y="3" size="0.8128" layer="25" font="vector" ratio="15">IC1=ATtiny25/45/85/13A</text>
 <wire x1="10.45" y1="4.1" x2="10.45" y2="5.1" width="0.2" layer="25"/>
 <wire x1="1.45" y1="1.2" x2="1.45" y2="2" width="0.4064" layer="25"/>
+<text x="19.5" y="5" size="0.8128" layer="29" font="vector" ratio="15">projects@carwe.de</text>
+<text x="19.5" y="6.5" size="0.8128" layer="29" font="vector" ratio="15">caphumidsens2 rev1</text>
 </plain>
 <attributes>
@@
 <attribute name="NAME" x="5.5" y="6" size="0.8128" layer="26" font="vector" ratio="20" rot="SMR270"/>
 </element>
-<element name="IC1" library="atmel" package="8S1" value="ATtiny25/45/85" x="4" y="5" smashed="yes">
+<element name="IC1" library="atmel" package="8S1" value="ATtiny25/45/85/13A" x="4" y="5" smashed="yes">
 <attribute name="OC_NEWARK" value="58M3773" x="21.78" y="1.19" size="1.778" layer="27" display="off"/>
 <attribute name="MPN" value="ATTINY13V-10SSU" x="21.78" y="1.19" size="1.778" layer="27" display="off"/>
@@
 </element>
 <element name="OSC1" library="seb" package="XO32" value="to be defined" x="11.9" y="3.5" rot="R90"/>
-<element name="R4" library="SparkFun" package="0805" value="to be defined" x="14.5" y="3.5" smashed="yes" rot="R90">
-<attribute name="NAME" x="15.362" y="1.9745" size="0.8128" layer="25" font="vector" ratio="15" rot="R180"/>
-<attribute name="VALUE" x="14.897" y="2.484" size="0.8128" layer="27" rot="R90"/>
+<element name="R4" library="SparkFun" package="0805" value="to be defined" x="14.7" y="3.5" smashed="yes" rot="R90">
+<attribute name="NAME" x="15.562" y="1.9745" size="0.8128" layer="25" font="vector" ratio="15" rot="R180"/>
+<attribute name="VALUE" x="15.097" y="2.484" size="0.8128" layer="27" rot="R90"/>
 </element>
 <element name="C3" library="SparkFun" package="0805" value="10n" x="9.5" y="3.4" smashed="yes" rot="R90">
@@
 <contactref element="OSC1" pad="2"/>
 <contactref element="OSC1" pad="2"/>
-<wire x1="13.5" y1="1.5" x2="16.5" y2="1.5" width="0.4064" layer="1"/>
+<wire x1="13.6" y1="1.5" x2="16.5" y2="1.5" width="0.4064" layer="1"/>
 <wire x1="16.5" y1="1.5" x2="17.5" y2="2.5" width="0.4064" layer="1"/>
 <wire x1="17.5" y1="2.5" x2="37" y2="2.5" width="0.4064" layer="1"/>
-<wire x1="12.5" y1="6.6" x2="13.5" y2="5.6" width="0.4064" layer="1"/>
-<wire x1="13.5" y1="5.6" x2="13.5" y2="1.5" width="0.4064" layer="1"/>
+<wire x1="12.5" y1="6.6" x2="13.6" y2="5.6" width="0.4064" layer="1"/>
+<wire x1="13.6" y1="5.6" x2="13.6" y2="1.5" width="0.4064" layer="1"/>
 <wire x1="6.2" y1="1.5" x2="6.7" y2="1.5" width="0.4064" layer="1"/>
 <wire x1="7.7" y1="1.5" x2="9.5" y2="1.5" width="0.4064" layer="1"/>
 <wire x1="6.7" y1="1.5" x2="7.7" y2="1.5" width="0.4064" layer="1"/>
 <wire x1="9.5" y1="1.5" x2="11.125" y2="1.5" width="0.4064" layer="1"/>
-<wire x1="11.125" y1="1.5" x2="13.5" y2="1.5" width="0.4064" layer="1"/>
+<wire x1="11.125" y1="1.5" x2="13.6" y2="1.5" width="0.4064" layer="1"/>
 <wire x1="6.2" y1="1.5" x2="5.895" y2="1.805" width="0.4064" layer="1"/>
 <wire x1="3" y1="2" x2="6.3" y2="2" width="0.4064" layer="16"/>
@@
 <wire x1="14.5" y1="8.4" x2="15.5" y2="8.4" width="0.4064" layer="1"/>
 <wire x1="4.625" y1="2.346" x2="4.625" y2="3.125" width="0.4064" layer="1"/>
-<wire x1="4.625" y1="3.125" x2="5.2" y2="3.7" width="0.4064" layer="1"/>
-<wire x1="5.2" y1="3.7" x2="7.1" y2="3.7" width="0.4064" layer="1"/>
-<wire x1="7.1" y1="3.7" x2="7.7" y2="4.3" width="0.4064" layer="1"/>
-<wire x1="15.5" y1="8.4" x2="16.746721875" y2="7.153278125" width="0.4064" layer="1"/>
-<wire x1="16.746721875" y1="7.153278125" x2="16.746721875" y2="5.953828125" width="0.4064" layer="1"/>
-<wire x1="16.746721875" y1="5.953828125" x2="16.29289375" y2="5.5" width="0.4064" layer="1"/>
-<wire x1="16.29289375" y1="5.5" x2="16.2" y2="5.5" width="0.4064" layer="1"/>
+<wire x1="4.625" y1="3.125" x2="5.15" y2="3.65" width="0.4064" layer="1"/>
+<wire x1="5.15" y1="3.65" x2="7.05" y2="3.65" width="0.4064" layer="1"/>
+<wire x1="7.05" y1="3.65" x2="7.7" y2="4.3" width="0.4064" layer="1"/>
 <via x="16.2" y="5.5" extent="1-16" drill="0.3302"/>
 <wire x1="16.2" y1="5.5" x2="6.8" y2="5.5" width="0.4064" layer="16"/>
@@
 <wire x1="6.8" y1="5.5" x2="7.7" y2="4.85" width="0.4064" layer="1"/>
 <wire x1="7.7" y1="4.85" x2="7.7" y2="4.3" width="0.4064" layer="1"/>
+<wire x1="16.2" y1="5.5" x2="16.6" y2="5.9" width="0.4064" layer="1"/>
+<wire x1="16.6" y1="5.9" x2="16.6" y2="7.3" width="0.4064" layer="1"/>
+<wire x1="16.6" y1="7.3" x2="15.5" y2="8.4" width="0.4064" layer="1"/>
 </signal>
 <signal name="SENSE_CAP">
@@
 <wire x1="6.7" y1="7.5" x2="5.905" y2="7.5" width="0.4064" layer="1"/>
 <wire x1="5.905" y1="7.5" x2="5.905" y2="7.654" width="0.4064" layer="1"/>
-<via x="15.6" y="2.6" extent="1-16" drill="0.3302"/>
-<wire x1="15.6" y1="2.6" x2="14.5" y2="2.6" width="0.4064" layer="1"/>
+<via x="15.8" y="2.6" extent="1-16" drill="0.3302"/>
+<wire x1="15.8" y1="2.6" x2="14.7" y2="2.6" width="0.4064" layer="1"/>
 <wire x1="17" y1="3.4" x2="16.2" y2="2.6" width="0.4064" layer="16"/>
-<wire x1="16.2" y1="2.6" x2="15.6" y2="2.6" width="0.4064" layer="16"/>
+<wire x1="16.2" y1="2.6" x2="15.8" y2="2.6" width="0.4064" layer="16"/>
 </signal>
 <signal name="CLOCK_IN">
@@
 <contactref element="R4" pad="2"/>
 <wire x1="15.6" y1="4.6" x2="6" y2="4.6" width="0.4064" layer="16"/>
-<wire x1="14.5" y1="4.4" x2="15.6" y2="4.4" width="0.4064" layer="1"/>
-<via x="15.6" y="4.4" extent="1-16" drill="0.3302"/>
-<wire x1="15.6" y1="4.4" x2="15.6" y2="4.6" width="0.4064" layer="16"/>
-<wire x1="6" y1="4.6" x2="5.54890625" y2="4.6" width="0.4064" layer="1"/>
-<wire x1="5.54890625" y1="4.6" x2="4.635" y2="5.51390625" width="0.4064" layer="1"/>
-<wire x1="4.635" y1="5.51390625" x2="4.635" y2="7.654" width="0.4064" layer="1"/>
+<wire x1="14.7" y1="4.4" x2="15.8" y2="4.4" width="0.4064" layer="1"/>
+<via x="15.8" y="4.4" extent="1-16" drill="0.3302"/>
+<wire x1="15.8" y1="4.4" x2="15.6" y2="4.6" width="0.4064" layer="16"/>
+<wire x1="6" y1="4.6" x2="4.635" y2="5.965" width="0.4064" layer="1"/>
+<wire x1="4.635" y1="5.965" x2="4.635" y2="7.654" width="0.4064" layer="1"/>
 <via x="6" y="4.6" extent="1-16" drill="0.3302"/>
 </signal>
