File: caphumidsens2_rev1_rc3.sch (EAGLE design)
At the start: 12 parts, among them IC1 ATtiny25/45/85

Commit message: finetuning, misc
Parts:
- IC1: value ATtiny25/45/85 -> ATtiny25/45/85/13A
Changed lines of the file:
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@@
 <part name="VCC" library="wirepad" deviceset="SMD2" device="" value="WIREPADSMD2,54-5,08"/>
 <part name="OUT" library="wirepad" deviceset="SMD2" device="" value="WIREPADSMD2,54-5,08"/>
-<part name="IC1" library="atmel" deviceset="TINY13" device="SSU" technology="V-10" value="ATtiny25/45/85"/>
+<part name="IC1" library="atmel" deviceset="TINY13" device="SSU" technology="V-10" value="ATtiny25/45/85/13A"/>
 <part name="P+5" library="supply1" deviceset="VCC" device=""/>
 <part name="GND5" library="supply1" deviceset="GND" device=""/>
